Commit message: fixing inertia value in shoulderpitch left, updating to use most recent hrl end-effector

File: hrl_gazebo_darci/urdf/A2R4_l_arm_defs.urdf.xacro (robot description, xacro)
@@ -51,5 +51,5 @@
         <inertia ixx="0.00074999"
                  iyy="0.00091729"
-                 izz="0.0083104"
+                 izz="0.00083104"
                  ixy="-0.00001075"
                  ixz="0.00002945"
@@ -166,36 +166,5 @@
 	      <origin xyz="0 0 0" rpy="0.0 0.0 0.0 " />
 	      <geometry name="wrist_LEFT_geom_collision">
-		      <mesh filename="package://${MESH_COLL}/A2R3/A2R3_T5_forearmRoll.stl" />
-	      </geometry>
-      </collision>
-    </link>
-    <!-- Darci Sleeve -->
-    <joint name="wrist_forearmor_joint" type="fixed">
-        <origin xyz="0.0 0.0 0.226" rpy="${-M_PI/2} 0 ${-M_PI/2}" />
-      <parent link="wrist_LEFT"/>
-      <child link="forearmor"/>
-    </joint>
-    <link name="forearmor">
-      <inertial>
-        <!-- mass, com, and I are all rough guess-timates -->
-        <origin xyz="0.0 0.0 -0.113" />
-        <mass value="0.5" />
-        <inertia ixx="0.0056125"
-                 iyy="0.0056125"
-                 izz="0.003725"
-                 ixy="1E-4"
-                 ixz="1E-5"
-                 iyz="1E-5" />
-      </inertial>
-      <visual>
-	    <origin xyz="0 0 0" rpy="0 0 0 " />
-	    <geometry name="wrist_LEFT_geom_forearmor">
-            <mesh filename="package://${MESH}/tactile_sensor/Darci_Forearmor.stl" />
-	    </geometry>
-      </visual>
-      <collision name="forearmor_collision">
-	      <origin xyz="0 0 0" rpy="0.0 0.0 0.0 " />
-	      <geometry name="wrist_LEFT_geom_collision_forearmor_front">
-              <mesh filename="package://${MESH_COLL}/tactile_sensor/Darci_Forearmor.stl"/>
+		      <mesh filename="package://${MESH_COLL}/A2R3/A2R3_T5_forearmRoll_coll.stl" />
 	      </geometry>
       </collision>
@@ -266,5 +235,6 @@
 	      <origin xyz="0 0 0" rpy="0.0 0.0 0.0 " />
 	      <geometry name="handmount_LEFT_geom_collision">
-		      <mesh filename="package://${MESH_COLL}/A2R3/A2R3_T7_wristYaw.stl" />
+		      <!--mesh filename="package://${MESH_COLL}/A2R3/A2R3_T7_wristYaw.stl" /-->
+                      <mesh filename="package://${MESH_COLL}/tactile_sensor/new_handmount_LEFT.stl"  scale="0.001 0.001 0.001"/>
 	      </geometry>
       </collision>
@@ -276,4 +246,5 @@
     </joint>
     <link name="handmount_FT_LEFT" >
+      <!-- values from data spec for ATI Mini40 sensor (read: should be fairly accurate)-->
       <inertial>
         <origin xyz="0.0 0.0 0.0" />
@@ -292,47 +263,54 @@
         </geometry>
       </visual>
-      <collision>
+      <!--collision>
 	    <origin xyz="0 0 0.0" rpy="0 0 0 " />
         <geometry>
             <cylinder radius="0.02" length="0.0125" />
         </geometry>
-      </collision>
+      </collision-->
     </link>
     <joint name="handmount_flipper_joint" type="fixed">
-        <origin xyz="0.0 0.0 -0.075" rpy="${-M_PI/2} 0 ${-M_PI/2}" />
+        <origin xyz="0.0 0.0 0.0" rpy="${-M_PI/2} 0 ${-M_PI/2}" />
       <parent link="handmount_FT_LEFT"/>
       <child link="flipper"/>
     </joint>
+    <!-- mass, com, inertia are all rough guess-timates -->
     <link name="flipper">
       <inertial>
-        <!-- mass, com, inertia are all rough guess-timates -->
-        <origin xyz="0.0 0.0 0.0" />
-        <mass value="0.75" />
-        <inertia ixx="0.02925"
-                 iyy="0.02925"
-                 izz="0.00225"
-                 ixy="1E-4"
-                 ixz="1E-4"
-                 iyz="1E-6" />
-      </inertial>
-      <visual>
-	    <origin xyz="0 0 0" rpy="0 0 0 " />
-	    <geometry name="flipper_geom">
-            <mesh filename="package://${MESH}/tactile_sensor/Darci_Flipper.stl"/>
+          <origin xyz="0.0 0.07 0.0"/>
+        <mass value="0.18"/>
+        <inertia ixx="0.00033755" ixy="0" ixz="0" iyy="0.00033755" iyz="0" izz="0.0001202"/>
+      </inertial>
+      <visual>
+        <origin rpy="0 0 0 " xyz="0 0 0"/>
+        <geometry name="flipper_geom">
+          <mesh filename="package://${MESH}/tactile_sensor/ee_simple.STL" scale="0.0009 0.00078 0.00085"/>
         </geometry>
-      </visual>
-      <collision name="flipper_collision">
-	    <origin xyz="0 0 0" rpy="0.0 0.0 0.0 " />
-	    <geometry name="wrist_LEFT_geom_collision_forearmor_front">
-            <mesh filename="package://${MESH_COLL}/tactile_sensor/Darci_Flipper.stl"/>
-	    </geometry>
-      </collision>
-    </link>
-    <joint name="handmount_flipper_tip_joint" type="fixed">
-        <origin xyz="0.0 0.0 -0.215" rpy="0 ${M_PI/2} 0" />
-      <parent link="handmount_FT_LEFT"/>
-      <child link="l_flipper_tip_frame"/>
-    </joint>
-    <link name="l_flipper_tip_frame" />
+        <material name="white">
+          <color rgba="1 1 1 1"/>
+        </material>
+      </visual>
+      <!--collision name="flipper_collision">
+        <origin rpy="0.0 0.0 0.0 " xyz="0 0 0"/>
+        <geometry name="flipper_geom_collision">
+          <mesh filename="package://${MESH_COLL}/tactile_sensor/ee_simple.STL" scale="0.0009 0.00078 0.0009"/>
+        </geometry>
+      </collision-->
+    </link>
+    <joint name="left_arm_ee" type="fixed">
+      <origin xyz="0 0 -0.17" rpy="-1.570796 0 0" />
+      <!--origin xyz="0 0 -0.19" rpy="-1.570796 0 0" /-->
+      <parent link="handmount_LEFT"/>
+      <child link="end_effector_LEFT"/>
+    </joint>
+    <link name="end_effector_LEFT">
+        <!--<inertial>
+        <mass value="0.093" />
+        <origin xyz="0 0 0" />
+        <inertia ixx="0.0" ixy="0.0" ixz="0.0"
+                 iyy="0.0" iyz="-0.0"
+                 izz="0.0" />
+         </inertial>-->
+    </link>
   </macro>
   <macro name="m3_l_arm" params="side parent reflect *origin">

File: hrl_gazebo_darci/urdf/gazebo/gazebo_links.urdf.xacro (robot description, xacro)
@@ -1,5 +1,5 @@
 <?xml version="1.0"?>
 <robot xmlns:xacro="http://www.ros.org/wiki/xacro">
-<!--  <macro name="surface_properties" params="link_name">
+<!--macro name="surface_properties" params="link_name">
     ##Example properties taken from Daehyung's pr2 contact params
     <gazebo reference="${link_name}_collision">
@@ -29,17 +29,32 @@
     <gazebo reference="${link_name}">
       <gravity>false</gravity>
-      <!--      <mu1>0.01</mu1>
+      <mu1>0.01</mu1>
+      <mu2>0.01</mu2>
+    </gazebo>
+  </macro>
+  <macro name="tactile_surface" params="link_name">
+    <gazebo reference="${link_name}">
+      <gravity>false</gravity>
+      <mu1>0.01</mu1>
+      <mu2>0.01</mu2>
+      <sensor name="${link_name}_tactile_sensor" type="contact">
+        <contact>
+          <collision>${link_name}_collision</collision>
+          <topic>__default_topic__</topic>
+        </contact>
+        <plugin name="ros_tactile_plugin_${link_name}" filename="libros_tactile_plugin.so" />
+        <always_on>1</always_on>
+        <update_rate>30.0</update_rate>
+        <visualize>false</visualize>
+      </sensor>
+    </gazebo>
+  </macro>
+  <!--  <macro name="tactile_surface_extended" params="link_name parent_link_name">
+    <gazebo reference="${link_name}">
+      <gravity>false</gravity>
+      <-      <mu1>0.01</mu1>
       <mu2>0.01</mu2>
       <kp>1E5</kp>
-      <kd>10</kd>-->
-    </gazebo>
-  </macro>
-  <macro name="tactile_surface" params="link_name parent_link_name">
-    <gazebo reference="${link_name}">
-      <gravity>false</gravity>
-      <!--      <mu1>0.01</mu1>
-      <mu2>0.01</mu2>
-      <kp>1E5</kp>
-      <kd>10</kd>-->
+      <kd>10</kd>->
       <sensor name="${link_name}_tactile_sensor" type="contact">
         <contact>
@@ -53,5 +68,5 @@
       </sensor>
     </gazebo>
-  </macro>
+</macro>-->
   <!-- BEGIN LEFT ARM -->
   <non_tactile_surface link_name="shoulderupper_LEFT"/>
@@ -59,10 +74,13 @@
   <non_tactile_surface link_name="bicep_LEFT"/>
   <non_tactile_surface link_name="elbowclevis_LEFT"/>
-  <non_tactile_surface link_name="wrist_LEFT"/>
-  <tactile_surface link_name="forearmor" parent_link_name="wrist_LEFT"/>
+  <!--surface_properties link_name="wrist_LEFT"/-->
+  <tactile_surface link_name="wrist_LEFT"/>
+  <!--tactile_surface link_name="forearmor" parent_link_name="wrist_LEFT"/-->
   <non_tactile_surface link_name="w_differential_LEFT"/>
-  <non_tactile_surface link_name="handmount_LEFT"/>
+  <tactile_surface link_name="handmount_LEFT"/>
   <non_tactile_surface link_name="handmount_FT_LEFT"/>
-  <tactile_surface link_name="flipper" parent_link_name="handmount_LEFT"/>
+  <non_tactile_surface link_name="flipper"/>
+  <!--tactile_surface_extended link_name="flipper" parent_link_name="handmount_LEFT"/-->
+  <!--surface_properties_extended link_name="flipper" parent_link_name="handmount_LEFT"/-->
   <!-- END LEFT ARM -->
   <!-- BEGIN RIGHT ARM -->

Commit message: merging changes from up to date hrl internal simulator package, including new arm controller gain files, and new meshes

File: hrl_gazebo_darci/urdf/A2R4_l_arm_defs.urdf.xacro (robot description, xacro)
@@ -305,11 +305,19 @@
     </joint>
     <link name="end_effector_LEFT">
-        <!--<inertial>
-        <mass value="0.093" />
-        <origin xyz="0 0 0" />
-        <inertia ixx="0.0" ixy="0.0" ixz="0.0"
-                 iyy="0.0" iyz="-0.0"
-                 izz="0.0" />
-         </inertial>-->
+        <!--inertial>
+          <mass value="0.093" />
+          <origin xyz="0 0 0" />
+          <inertia ixx="0.0" ixy="0.0" ixz="0.0"
+                   iyy="0.0" iyz="-0.0"
+                   izz="0.0" />
+          </inertial-->
+          <visual>
+            <geometry>
+              <cylinder radius="0.001" length="0.01" />
+            </geometry>
+            <material name="white">
+              <color rgba="1 1 1 1"/>
+            </material>
+          </visual>
     </link>
   </macro>
