Commit message: dummy file for simco.urdf.xacro, pulling hrl specific content out of arm file. added new ee file for hrl end effector.

File: gt_meka_description/urdf/A2R4_l_arm_defs.urdf.xacro (robot description, xacro)
@@ -166,5 +166,6 @@
 	      <origin xyz="0 0 0" rpy="0.0 0.0 0.0 " />
 	      <geometry name="wrist_LEFT_geom_collision">
-		      <mesh filename="package://${MESH_COLL}/A2R3/A2R3_T5_forearmRoll_coll.stl" />
+		      <mesh filename="package://${MESH_COLL}/A2R3/A2R3_T5_forearmRoll.stl" />
+              <!--mesh filename="package://${MESH_COLL}/A2R3/A2R3_T5_forearmRoll_coll.stl"/ -->
 	      </geometry>
       </collision>
@@ -235,89 +236,8 @@
 	      <origin xyz="0 0 0" rpy="0.0 0.0 0.0 " />
 	      <geometry name="handmount_LEFT_geom_collision">
-		      <!--mesh filename="package://${MESH_COLL}/A2R3/A2R3_T7_wristYaw.stl" /-->
-                      <mesh filename="package://${MESH_COLL}/tactile_sensor/new_handmount_LEFT.stl"  scale="0.001 0.001 0.001"/>
-	      </geometry>
-      </collision>
-    </link>
-    <joint name="handmount_ft_joint" type="fixed">
-        <origin xyz="0.0 0.0 -0.05125" rpy="0 0 0" />
-      <parent link="handmount_LEFT"/>
-      <child link="handmount_FT_LEFT"/>
-    </joint>
-    <link name="handmount_FT_LEFT" >
-      <!-- values from data spec for ATI Mini40 sensor (read: should be fairly accurate)-->
-      <inertial>
-        <origin xyz="0.0 0.0 0.0" />
-        <mass value="0.0499" />
-        <inertia ixx="3.3838E-6"
-                 iyy="3.3838E-6"
-                 izz="1E-7"
-                 ixy="0"
-                 ixz="0"
-                 iyz="0" />
-      </inertial>
-      <visual>
-	    <origin xyz="0 0 0.0" rpy="0 0 0 " />
-        <geometry>
-            <cylinder radius="0.02" length="0.0125" />
-        </geometry>
-      </visual>
-      <!--collision>
-	    <origin xyz="0 0 0.0" rpy="0 0 0 " />
-        <geometry>
-            <cylinder radius="0.02" length="0.0125" />
-        </geometry>
-      </collision-->
-    </link>
-    <joint name="handmount_flipper_joint" type="fixed">
-        <origin xyz="0.0 0.0 0.0" rpy="${-M_PI/2} 0 ${-M_PI/2}" />
-      <parent link="handmount_FT_LEFT"/>
-      <child link="flipper"/>
-    </joint>
-    <!-- mass, com, inertia are all rough guess-timates -->
-    <link name="flipper">
-      <inertial>
-          <origin xyz="0.0 0.07 0.0"/>
-        <mass value="0.18"/>
-        <inertia ixx="0.00033755" ixy="0" ixz="0" iyy="0.00033755" iyz="0" izz="0.0001202"/>
-      </inertial>
-      <visual>
-        <origin rpy="0 0 0 " xyz="0 0 0"/>
-        <geometry name="flipper_geom">
-          <mesh filename="package://${MESH}/tactile_sensor/ee_simple.STL" scale="0.0009 0.00078 0.00085"/>
-        </geometry>
-        <material name="white">
-          <color rgba="1 1 1 1"/>
-        </material>
-      </visual>
-      <!--collision name="flipper_collision">
-        <origin rpy="0.0 0.0 0.0 " xyz="0 0 0"/>
-        <geometry name="flipper_geom_collision">
-          <mesh filename="package://${MESH_COLL}/tactile_sensor/ee_simple.STL" scale="0.0009 0.00078 0.0009"/>
-        </geometry>
-      </collision-->
-    </link>
-    <joint name="left_arm_ee" type="fixed">
-      <origin xyz="0 0 -0.17" rpy="-1.570796 0 0" />
-      <!--origin xyz="0 0 -0.19" rpy="-1.570796 0 0" /-->
-      <parent link="handmount_LEFT"/>
-      <child link="end_effector_LEFT"/>
-    </joint>
-    <link name="end_effector_LEFT">
-        <!--inertial>
-          <mass value="0.093" />
-          <origin xyz="0 0 0" />
-          <inertia ixx="0.0" ixy="0.0" ixz="0.0"
-                   iyy="0.0" iyz="-0.0"
-                   izz="0.0" />
-          </inertial-->
-          <visual>
-            <geometry>
-              <cylinder radius="0.001" length="0.01" />
-            </geometry>
-            <material name="white">
-              <color rgba="1 1 1 1"/>
-            </material>
-          </visual>
+		      <mesh filename="package://${MESH_COLL}/A2R3/A2R3_T7_wristYaw.stl" />
+              <!--mesh filename="package://${MESH_COLL}/tactile_sensor/new_handmount_LEFT.stl"  scale="0.001 0.001 0.001"/-->
+	      </geometry>
+      </collision>
     </link>
   </macro>

File: gt_meka_description/urdf/simco.urdf.xacro (robot description, xacro)
@@ -6,6 +6,7 @@
 <!-- simulator_gazebo plugins and tags for inclusion in sdf -->
   <include filename="./gazebo/gazebo.urdf.xacro" />
-  <include filename="./gazebo/gazebo_joints.urdf.xacro" />
-  <include filename="./gazebo/gazebo_links.urdf.xacro" />
+  <!-- Additional gazebo files added for creating tactile sensors on some links for HRL -->
+  <!--  <include filename="./gazebo/gazebo_joints.urdf.xacro" />
+  <include filename="./gazebo/gazebo_links.urdf.xacro" />-->
 <!-- Meka Base -->
   <include filename="./B1R2B_defs.urdf.xacro" />
@@ -15,6 +16,4 @@
   <include filename="./A2R4_r_arm_defs.urdf.xacro" />
   <include filename="./A2R4_l_arm_defs.urdf.xacro" />
-<!-- HRL End Effector -->
-  <include filename="./HRL_EE_Left.urdf.xacro" />
   <!-- john added transmissions -->
   <include filename="./transmissions/A2R4_r_arm_defs.transmission.xacro" />
@@ -65,7 +64,4 @@
       <origin xyz="0.0 0.18465 0." rpy="0.0 0.0 0.0" />
   </m3_l_arm>
-  <HRL_EE_Left side="l" reflect="-1" parent="handmount_LEFT">
-      <origin xyz="0.0 0.0 -0.05125" rpy="0 0 0" />
-  </HRL_EE_Left>
   <!-- john added transmissions -->
   <m3_zlift_transmission name="torso_lift"/>
