Commit message: Added tabletop, moved asus launch files, and gave head control

File: gt_meka_description/urdf/simco-groovy.urdf.xacro (robot description, xacro)
@@ -10,4 +10,5 @@
   <include filename="./gazebo/gazebo_joints.urdf.xacro" />
   <include filename="./gazebo/gazebo_hand_joints.urdf.xacro" />
+  <include filename="./gazebo/gazebo_head_joints.urdf.xacro" />
   <!--include filename="./gazebo/gazebo_links.urdf.xacro" /-->
   <!--include filename="./gazebo/gazebo_hand_links.urdf.xacro" /-->
@@ -28,19 +29,6 @@
   <include filename="./transmissions/A2R4_l_arm_defs.transmission.xacro" />
   <include filename="./transmissions/zlift_defs.transmission.xacro" />
+  <include filename="./transmissions/SIMC_head_defs.transmission.xacro" />
   <link name="world" />
-  <!-- Added in as test -->
-  <!--link name="base_link">
-     <inertial>
-          <mass value="1" />
-          <origin xyz="0 0 0" />
-          <inertia ixx="0"  ixy="0"  ixz="0" iyy="0"  iyz="0" izz="0" />
-     </inertial>
-  </link-->
-  <!-- Solid Base -->
-  <!--joint name="base_joint" type="fixed">
-      <origin xyz="0 0 0" rpy="0 0 0" />
-    <parent link="world" />
-    <child link="base_link" />
-  </joint-->
   <meka_base reflect="1" parent="world">
     <origin xyz="0.0 0.0 0.02" rpy="0 0 0" />
@@ -103,3 +91,4 @@
   <m3_r_arm_transmission side="r" reflect="1" parent="torso_lift_link"/>
   <m3_l_arm_transmission side="l" reflect="1" parent="torso_lift_link"/>
+  <m3_head_transmission />
 </robot>

File: gt_meka_description/urdf/simco.urdf.xacro (robot description, xacro)
@@ -9,4 +9,5 @@
   <include filename="./gazebo/gazebo_joints.urdf.xacro" />
   <include filename="./gazebo/gazebo_hand_joints.urdf.xacro" />
+  <include filename="./gazebo/gazebo_head_joints.urdf.xacro" />
   <!--include filename="./gazebo/gazebo_links.urdf.xacro" /-->
   <!--include filename="./gazebo/gazebo_hand_links.urdf.xacro" /-->
@@ -24,22 +25,9 @@
   <include filename="./SIMC_head_defs.urdf.xacro" />
   <!-- john added transmissions -->
-  <include filename="./transmissions/A2R4_r_arm_defs.transmission.xacro" />
-  <include filename="./transmissions/A2R4_l_arm_defs.transmission.xacro" />
-  <include filename="./transmissions/zlift_defs.transmission.xacro" />
+  <include filename="./transmissions_hydro/A2R4_r_arm_defs.transmission.xacro" />
+  <include filename="./transmissions_hydro/A2R4_l_arm_defs.transmission.xacro" />
+  <include filename="./transmissions_hydro/zlift_defs.transmission.xacro" />
+  <include filename="./transmissions_hydro/SIMC_head_defs.transmission.xacro" />
   <link name="world" />
-  <!-- Added in as test -->
-  <!--link name="base_link">
-     <inertial>
-          <mass value="1" />
-          <origin xyz="0 0 0" />
-          <inertia ixx="0"  ixy="0"  ixz="0" iyy="0"  iyz="0" izz="0" />
-     </inertial>
-  </link-->
-  <!-- Solid Base -->
-  <!--joint name="base_joint" type="fixed">
-      <origin xyz="0 0 0" rpy="0 0 0" />
-    <parent link="world" />
-    <child link="base_link" />
-  </joint-->
   <meka_base reflect="1" parent="world">
     <origin xyz="0.0 0.0 0.02" rpy="0 0 0" />
@@ -102,3 +90,4 @@
   <m3_r_arm_transmission side="r" reflect="1" parent="torso_lift_link"/>
   <m3_l_arm_transmission side="l" reflect="1" parent="torso_lift_link"/>
+  <m3_head_transmission />
 </robot>

Commit message: added in more edits for arm and hand control

File: gt_meka_description/urdf/simco-groovy.urdf.xacro (robot description, xacro)
@@ -37,6 +37,6 @@
   </meka_base>
   <meka_zlift  side="r" reflect="1" parent="dummy_3">
-    <!--origin xyz="0.42 0.0 0.6137" rpy="0 0 0" /-->
-    <origin xyz="0.42 0.0 0.85" rpy="0 0 0" />
+    <origin xyz="0.42 0.0 0.6137" rpy="0 0 0" />
+    <!--origin xyz="0.42 0.0 0.85" rpy="0 0 0" /-->
   </meka_zlift>
   <!-- Torso -->
