Commit message: added in files for getting the real robot to run

File: gt_meka_description/urdf/Z1R2B_defs.urdf.xacro (robot description, xacro)
@@ -4,14 +4,17 @@
   <macro name="meka_zlift" params="side parent reflect *origin">
     <!-- Shoulder pan -->
-    <joint name="torso_lift_joint" type="prismatic">
+    <!--joint name="torso_lift_joint" type="prismatic"-->
+    <joint name="zlift_joint" type="prismatic">
       <axis xyz="0 0 1" />
       <insert_block name="origin" />
       <parent link="${parent}"/>
-      <child link="torso_lift_link"/>
+      <!--child link="torso_lift_link"/-->
+      <child link="zlift_link"/>
       <!-- torso_lift limit values are purely invented -->
       <limit lower="0.0"  upper="0.7" velocity="0.2" effort="2000.0"/>
       <dynamics damping="100.0" />
     </joint>
-    <link name="torso_lift_link">
+    <!--link name="torso_lift_link"-->
+    <link name="zlift_link">
       <inertial>
         <mass value="5.799322" />

File: gt_meka_description/urdf/simco-groovy.urdf.xacro (robot description, xacro)
@@ -43,5 +43,6 @@
   <joint name="chest_joint" type="fixed">
       <origin xyz="0.0 0.0 0.0"/>
-    <parent link="torso_lift_link" />
+    <!--parent link="torso_lift_link" /-->
+    <parent link="zlift_link" />
     <child link="chest_link" />
   </joint>
@@ -71,8 +72,10 @@
   </link>
   <!-- Add Arms -->
-  <m3_r_arm side="r" reflect="1" parent="torso_lift_link">
+  <!--m3_r_arm side="r" reflect="1" parent="torso_lift_link"-->
+  <m3_r_arm side="r" reflect="1" parent="zlift_link">
       <origin xyz="0.0 -0.18465 0" rpy="0.0 0.0 0.0" />
   </m3_r_arm>
-  <m3_l_arm side="l" reflect="-1" parent="torso_lift_link">
+  <!--m3_l_arm side="l" reflect="-1" parent="torso_lift_link"-->
+  <m3_l_arm side="l" reflect="-1" parent="zlift_link">
       <origin xyz="0.0 0.18465 0" rpy="0.0 0.0 0.0" />
   </m3_l_arm>
@@ -89,5 +92,6 @@
   </m3_head>
   <!-- john added transmissions -->
-  <m3_zlift_transmission name="torso_lift"/>
+  <!--m3_zlift_transmission name="torso_lift"/-->
+  <m3_zlift_transmission name="zlift"/>
   <m3_r_arm_transmission side="r" reflect="1" parent="torso_lift_link"/>
   <m3_l_arm_transmission side="l" reflect="1" parent="torso_lift_link"/>

Commit message: working modified curi description with zlift mods

File: gt_meka_description/urdf/Z1R2B_defs.urdf.xacro (robot description, xacro)
@@ -4,17 +4,17 @@
   <macro name="meka_zlift" params="side parent reflect *origin">
     <!-- Shoulder pan -->
-    <!--joint name="torso_lift_joint" type="prismatic"-->
-    <joint name="zlift_joint" type="prismatic">
+    <joint name="torso_lift_joint" type="prismatic">
+    <!--joint name="zlift_joint" type="prismatic"-->
       <axis xyz="0 0 1" />
       <insert_block name="origin" />
       <parent link="${parent}"/>
-      <!--child link="torso_lift_link"/-->
-      <child link="zlift_link"/>
+      <child link="torso_lift_link"/>
+      <!--child link="zlift_link"/-->
       <!-- torso_lift limit values are purely invented -->
       <limit lower="0.0"  upper="0.7" velocity="0.2" effort="2000.0"/>
       <dynamics damping="100.0" />
     </joint>
-    <!--link name="torso_lift_link"-->
-    <link name="zlift_link">
+    <link name="torso_lift_link">
+    <!--link name="zlift_link"-->
       <inertial>
         <mass value="5.799322" />

File: gt_meka_description/urdf/simco-groovy.urdf.xacro (robot description, xacro)
@@ -43,6 +43,6 @@
   <joint name="chest_joint" type="fixed">
       <origin xyz="0.0 0.0 0.0"/>
-    <!--parent link="torso_lift_link" /-->
-    <parent link="zlift_link" />
+    <parent link="torso_lift_link" />
+    <!--parent link="zlift_link" /-->
     <child link="chest_link" />
   </joint>
@@ -72,10 +72,10 @@
   </link>
   <!-- Add Arms -->
-  <!--m3_r_arm side="r" reflect="1" parent="torso_lift_link"-->
-  <m3_r_arm side="r" reflect="1" parent="zlift_link">
+  <m3_r_arm side="r" reflect="1" parent="torso_lift_link">
+  <!--m3_r_arm side="r" reflect="1" parent="zlift_link"-->
       <origin xyz="0.0 -0.18465 0" rpy="0.0 0.0 0.0" />
   </m3_r_arm>
-  <!--m3_l_arm side="l" reflect="-1" parent="torso_lift_link"-->
-  <m3_l_arm side="l" reflect="-1" parent="zlift_link">
+  <m3_l_arm side="l" reflect="-1" parent="torso_lift_link">
+  <!--m3_l_arm side="l" reflect="-1" parent="zlift_link"-->
       <origin xyz="0.0 0.18465 0" rpy="0.0 0.0 0.0" />
   </m3_l_arm>
@@ -92,6 +92,6 @@
   </m3_head>
   <!-- john added transmissions -->
-  <!--m3_zlift_transmission name="torso_lift"/-->
-  <m3_zlift_transmission name="zlift"/>
+  <m3_zlift_transmission name="torso_lift"/>
+  <!--m3_zlift_transmission name="zlift"/-->
   <m3_r_arm_transmission side="r" reflect="1" parent="torso_lift_link"/>
   <m3_l_arm_transmission side="l" reflect="1" parent="torso_lift_link"/>
