Commit message: Added some controller and urdf changes to work with all parts of the head and to publish the hands

File: gt_meka_description/urdf/SIMC_head_defs.urdf.xacro (robot description, xacro)
@@ -129,5 +129,5 @@
       </collision>
     </link>
-    <!--joint name="head_j4" type="revolute">
+    <joint name="head_j4" type="revolute">
 	  <axis xyz="0 -1 0" />
       <limit effort="100" velocity="${1600*M_PI/180}" lower="${-70.1*M_PI/180}" upper="${70.1*M_PI/180}" />
@@ -207,5 +207,7 @@
       </collision>
     </link>
-    <joint name="head_j7_rt_eyelid_top" type="revolute">
+    <!--joint name="head_j7_rt_eyelid_top" type="revolute"-->
+    <!-- temp hack since real robot doesn't support anything other than joint 7 currently-->
+    <joint name="head_j7" type="revolute">
 	    <axis xyz="0 -1 0" />
       <limit effort="100" velocity="${1600*M_PI/180}" lower="${2.0*M_PI/180}" upper="${68.0*M_PI/180}" />
@@ -414,5 +416,5 @@
 	      </geometry>
       </collision>
-    </link-->
+    </link>
 </macro>
   <macro name="m3_head" params="side parent reflect *origin">

File: gt_meka_description/urdf/gazebo/gazebo_head_joints.urdf.xacro (robot description, xacro)
@@ -56,4 +56,13 @@
   </gazebo>
   <gazebo reference="head_j6">
+    <kp>1.0</kp>
+    <kd>1.0</kd>
+    <stopCfm>0.8</stopCfm>
+    <stopErp>0.5</stopErp>
+    <provideFeedback>true</provideFeedback>
+    <cfmDamping>true</cfmDamping>
+    <fudgeFactor>0.0</fudgeFactor>
+  </gazebo>
+  <gazebo reference="head_j7">
     <kp>1.0</kp>
     <kd>1.0</kd>

File: gt_meka_description/urdf/transmissions/SIMC_head_defs.transmission.xacro (robot description, xacro)
@@ -42,9 +42,15 @@
     <mechanicalReduction>1</mechanicalReduction>
   </transmission>
-  <transmission name="head_t7_rt_eyelid_top" type="pr2_mechanism_model/SimpleTransmission">
+  <!-- Temp for gazebo -->
+  <transmission name="head_t7" type="pr2_mechanism_model/SimpleTransmission">
+      <actuator name="head_a7"/>
+      <joint name="head_j7"/>
+    <mechanicalReduction>1</mechanicalReduction>
+  </transmission>
+  <!--transmission name="head_t7_rt_eyelid_top" type="pr2_mechanism_model/SimpleTransmission">
       <actuator name="head_a7_rt_eyelid_top"/>
       <joint name="head_j7_rt_eyelid_top"/>
     <mechanicalReduction>1</mechanicalReduction>
-  </transmission>
+  </transmission-->
   <transmission name="head_t7_rt_eyelid_bottom" type="pr2_mechanism_model/SimpleTransmission">
       <actuator name="head_a7_rt_eyelid_bottom"/>
@@ -87,6 +93,6 @@
   <macro name="m3_head_transmission">
     <m3_neck_transmission/>
-    <!--m3_eye_transmission/>
-    <m3_ear_transmission/-->
+    <m3_eye_transmission/>
+    <m3_ear_transmission/>
   </macro>
 </robot>
