Commit message: forgot to commit the modified files for hydro curi

File: gt_meka_description/urdf/SIMC_head_defs.urdf.xacro (robot description, xacro)
@@ -140,5 +140,5 @@
         <mass value="0.01" />
         <origin xyz="0.0 0.0 0.0" rpy="0 0 0" />
-        <inertia ixx="0" ixy="0" ixz="0" iyy="0" iyz="0" izz="0" />
+        <inertia ixx="0.01" ixy="0" ixz="0" iyy="0.01" iyz="0" izz="0.01" />
       </inertial>
       <visual>
@@ -166,5 +166,5 @@
         <mass value="0.01" />
         <origin xyz="0.0 0.0 0.0" rpy="0 0 0" />
-        <inertia ixx="0" ixy="0" ixz="0" iyy="0" iyz="0" izz="0" />
+        <inertia ixx="0.01" ixy="0" ixz="0" iyy="0.01" iyz="0" izz="0.01" />
       </inertial>
       <visual>
@@ -192,5 +192,5 @@
         <mass value="0.01" />
         <origin xyz="0.0 0.0 0.0" rpy="0 0 0" />
-        <inertia ixx="0" ixy="0" ixz="0" iyy="0" iyz="0" izz="0" />
+        <inertia ixx="0.01" ixy="0" ixz="0" iyy="0.01" iyz="0" izz="0.01" />
       </inertial>
       <visual>
@@ -220,5 +220,5 @@
         <mass value="0.01" />
         <origin xyz="0.0 0.0 0.0" rpy="0 0 0" />
-        <inertia ixx="0" ixy="0" ixz="0" iyy="0" iyz="0" izz="0" />
+        <inertia ixx="0.01" ixy="0" ixz="0" iyy="0.01" iyz="0" izz="0.01" />
       </inertial>
       <visual>
@@ -246,5 +246,5 @@
         <mass value="0.01" />
         <origin xyz="0.0 0.0 0.0" rpy="0 0 0" />
-        <inertia ixx="0" ixy="0" ixz="0" iyy="0" iyz="0" izz="0" />
+        <inertia ixx="0.01" ixy="0" ixz="0" iyy="0.01" iyz="0" izz="0.01" />
       </inertial>
       <visual>
@@ -272,5 +272,5 @@
         <mass value="0.01" />
         <origin xyz="0.0 0.0 0.0" rpy="0 0 0" />
-        <inertia ixx="0" ixy="0" ixz="0" iyy="0" iyz="0" izz="0" />
+        <inertia ixx="0.01" ixy="0" ixz="0" iyy="0.01" iyz="0" izz="0.01" />
       </inertial>
       <visual>
@@ -298,5 +298,5 @@
         <mass value="0.01" />
         <origin xyz="0.0 0.0 0.0" rpy="0 0 0" />
-        <inertia ixx="0" ixy="0" ixz="0" iyy="0" iyz="0" izz="0" />
+        <inertia ixx="0.01" ixy="0" ixz="0" iyy="0.01" iyz="0" izz="0.01" />
       </inertial>
       <visual>
@@ -324,5 +324,5 @@
         <mass value="0.01" />
         <origin xyz="0.0 0.0 0.0" rpy="0 0 0" />
-        <inertia ixx="0" ixy="0" ixz="0" iyy="0" iyz="0" izz="0" />
+        <inertia ixx="0.01" ixy="0" ixz="0" iyy="0.01" iyz="0" izz="0.01" />
       </inertial>
       <visual>
@@ -350,5 +350,5 @@
         <mass value="0.01" />
         <origin xyz="0.0 0.0 0.0" rpy="0 0 0" />
-        <inertia ixx="0" ixy="0" ixz="0" iyy="0" iyz="0" izz="0" />
+        <inertia ixx="0.01" ixy="0" ixz="0" iyy="0.01" iyz="0" izz="0.01" />
       </inertial>
       <visual>
@@ -376,5 +376,5 @@
         <mass value="0.01" />
         <origin xyz="0.0 0.0 0.0" rpy="0 0 0" />
-        <inertia ixx="0" ixy="0" ixz="0" iyy="0" iyz="0" izz="0" />
+        <inertia ixx="0.01" ixy="0" ixz="0" iyy="0.01" iyz="0" izz="0.01" />
       </inertial>
       <visual>
@@ -402,5 +402,5 @@
         <mass value="0.01" />
         <origin xyz="0.0 0.0 0.0" rpy="0 0 0" />
-        <inertia ixx="0" ixy="0" ixz="0" iyy="0" iyz="0" izz="0" />
+        <inertia ixx="0.01" ixy="0" ixz="0" iyy="0.01" iyz="0" izz="0.01" />
       </inertial>
       <visual>

File: gt_meka_description/urdf/gazebo/gazebo.urdf.xacro (robot description, xacro)
@@ -5,4 +5,9 @@
       <plugin name="ros_model_plugin" filename="libros_model_plugin.so" />
       <static> false </static>
+  <plugin name="gazebo_ros_control" filename="libgazebo_ros_control.so">
+    <!--robotNamespace>curi</robotNamespace-->
+    <robotNamespace></robotNamespace>
+    <robotSimType>gazebo_ros_control/DefaultRobotHWSim</robotSimType>
+  </plugin>
   </gazebo>
 </robot>

File: gt_meka_description/urdf/simco.urdf.xacro (robot description, xacro)
@@ -25,8 +25,10 @@
   <include filename="./SIMC_head_defs.urdf.xacro" />
   <!-- john added transmissions -->
+  <include filename="./transmissions_hydro/zlift_defs.transmission.xacro" />
   <include filename="./transmissions_hydro/A2R4_r_arm_defs.transmission.xacro" />
   <include filename="./transmissions_hydro/A2R4_l_arm_defs.transmission.xacro" />
-  <include filename="./transmissions_hydro/zlift_defs.transmission.xacro" />
   <include filename="./transmissions_hydro/SIMC_head_defs.transmission.xacro" />
+  <include filename="./transmissions_hydro/H2R4_r_hand_defs.transmission.xacro" />
+  <include filename="./transmissions_hydro/H2R4_l_hand_defs.transmission.xacro" />
   <link name="world" />
   <meka_base reflect="1" parent="world">
@@ -35,4 +37,5 @@
   <meka_zlift  side="r" reflect="1" parent="dummy_3">
     <origin xyz="0.42 0.0 0.6137" rpy="0 0 0" />
+    <!--origin xyz="0.42 0.0 0.85" rpy="0 0 0" /-->
   </meka_zlift>
   <!-- Torso -->
@@ -40,4 +43,5 @@
       <origin xyz="0.0 0.0 0.0"/>
     <parent link="torso_lift_link" />
+    <!--parent link="zlift_link" /-->
     <child link="chest_link" />
   </joint>
@@ -74,12 +78,10 @@
   </m3_l_arm>
   <!-- Add Hands -->
-  <!--
   <m3_r_hand side="r" reflect="1" parent="handmount_RIGHT">
     <origin xyz="0.0 0.0 0.0" rpy="0 0 0" />
   </m3_r_hand>
-  <m3_l_hand side="l" reflect="1" parent="handmount_LEFT">
+  <m3_l_hand side="l" reflect="-1" parent="handmount_LEFT">
     <origin xyz="0.0 0.0 0.0" rpy="0 0 0" />
   </m3_l_hand>
-  -->
   <!-- Add Head -->
   <m3_head side="r" reflect="1" parent="chest_link">
@@ -91,3 +93,5 @@
   <m3_l_arm_transmission side="l" reflect="1" parent="torso_lift_link"/>
   <m3_head_transmission />
+  <m3_r_hand_transmission />
+  <m3_l_hand_transmission />
 </robot>

File: gt_meka_description/urdf/transmissions_hydro/A2R4_l_arm_defs.transmission.xacro (robot description, xacro)
@@ -9,4 +9,5 @@
         <hardwareInterface>PositionJointInterface</hardwareInterface>
         <mechanicalReduction>1.0</mechanicalReduction>
+      </actuator>
     </transmission>
     <!-- Shoulder lift -->
@@ -17,38 +18,54 @@
         <hardwareInterface>PositionJointInterface</hardwareInterface>
         <mechanicalReduction>1.0</mechanicalReduction>
+      </actuator>
     </transmission>
     <!-- Upperarm roll: internal fixed attchment point for upper arm -->
-    <transmission name="left_arm_t2" type="pr2_mechanism_model/SimpleTransmission">
-      <actuator name="left_arm_a2" />
+    <transmission name="left_arm_t2">
+      <type>transmission_interface/SimpleTransmission</type>
       <joint name="left_arm_j2" />
-      <mechanicalReduction>1.0</mechanicalReduction>
+      <actuator name="left_arm_a2">
+        <hardwareInterface>PositionJointInterface</hardwareInterface>
+        <mechanicalReduction>1.0</mechanicalReduction>
+      </actuator>
     </transmission>
   </macro>
   <!-- ============================   Upper Arm   ============================ -->
   <macro name="m3_l_upper_arm_transmission" params="side parent reflect">
-    <transmission name="left_arm_t3" type="pr2_mechanism_model/SimpleTransmission">
-      <actuator name="left_arm_a3" />
+    <transmission name="left_arm_t3">
+      <type>transmission_interface/SimpleTransmission</type>
       <joint name="left_arm_j3" />
-      <mechanicalReduction>1.0</mechanicalReduction>
+      <actuator name="left_arm_a3">
+        <hardwareInterface>PositionJointInterface</hardwareInterface>
+        <mechanicalReduction>1.0</mechanicalReduction>
+      </actuator>
     </transmission>
     <!-- Elbow flex -->
-    <transmission name="left_arm_t4" type="pr2_mechanism_model/SimpleTransmission">
-      <actuator name="left_arm_a4" />
+    <transmission name="left_arm_t4">
+      <type>transmission_interface/SimpleTransmission</type>
       <joint name="left_arm_j4" />
-      <mechanicalReduction>1.0</mechanicalReduction>
+      <actuator name="left_arm_a4">
+        <hardwareInterface>PositionJointInterface</hardwareInterface>
+        <mechanicalReduction>1.0</mechanicalReduction>
+      </actuator>
     </transmission>
   </macro>
   <!-- ============================   Forearm   ============================ -->
   <macro name="m3_l_forearm_transmission" params="side parent reflect">
-    <transmission name="left_arm_t5" type="pr2_mechanism_model/SimpleTransmission">
-      <actuator name="left_arm_a5" />
+    <transmission name="left_arm_t5">
+      <type>transmission_interface/SimpleTransmission</type>
       <joint name="left_arm_j5" />
-      <mechanicalReduction>1.0</mechanicalReduction>
+      <actuator name="left_arm_a5">
+        <hardwareInterface>PositionJointInterface</hardwareInterface>
+        <mechanicalReduction>1.0</mechanicalReduction>
+      </actuator>
     </transmission>
     <!-- Wrist flex -->
-    <transmission name="left_arm_t6" type="pr2_mechanism_model/SimpleTransmission">
-      <actuator name="left_arm_a6" />
+    <transmission name="left_arm_t6">
+      <type>transmission_interface/SimpleTransmission</type>
       <joint name="left_arm_j6" />
-      <mechanicalReduction>1.0</mechanicalReduction>
+      <actuator name="left_arm_a6">
+        <hardwareInterface>PositionJointInterface</hardwareInterface>
+        <mechanicalReduction>1.0</mechanicalReduction>
+      </actuator>
     </transmission>
   </macro>

File: gt_meka_description/urdf/transmissions_hydro/A2R4_r_arm_defs.transmission.xacro (robot description, xacro)
@@ -3,48 +3,69 @@
   <macro name="m3_r_shoulder_transmission" params="side parent reflect">
     <!-- Shoulder pan -->
-    <transmission name="right_arm_t0" type="pr2_mechanism_model/SimpleTransmission">
-      <actuator name="right_arm_a0" />
+    <transmission name="right_arm_t0">
+      <type>transmission_interface/SimpleTransmission</type>
       <joint name="right_arm_j0" />
-      <mechanicalReduction>1.0</mechanicalReduction>
+      <actuator name="right_arm_a0">
+        <hardwareInterface>PositionJointInterface</hardwareInterface>
+        <mechanicalReduction>1.0</mechanicalReduction>
+      </actuator>
     </transmission>
     <!-- Shoulder lift -->
-    <transmission name="right_arm_t1" type="pr2_mechanism_model/SimpleTransmission">
-      <actuator name="right_arm_a1" />
+    <transmission name="right_arm_t1">
+      <type>transmission_interface/SimpleTransmission</type>
       <joint name="right_arm_j1" />
-      <mechanicalReduction>1.0</mechanicalReduction>
+      <actuator name="right_arm_a1">
+        <hardwareInterface>PositionJointInterface</hardwareInterface>
+        <mechanicalReduction>1.0</mechanicalReduction>
+      </actuator>
     </transmission>
     <!-- Upperarm roll: internal fixed attchment point for upper arm -->
-    <transmission name="right_arm_t2" type="pr2_mechanism_model/SimpleTransmission">
-      <actuator name="right_arm_a2" />
+    <transmission name="right_arm_t2">
+      <type>transmission_interface/SimpleTransmission</type>
       <joint name="right_arm_j2" />
-      <mechanicalReduction>1.0</mechanicalReduction>
+      <actuator name="right_arm_a2">
+        <hardwareInterface>PositionJointInterface</hardwareInterface>
+        <mechanicalReduction>1.0</mechanicalReduction>
+      </actuator>
     </transmission>
   </macro>
   <!-- ============================   Upper Arm   ============================ -->
   <macro name="m3_r_upper_arm_transmission" params="side parent reflect">
-    <transmission name="right_arm_t3" type="pr2_mechanism_model/SimpleTransmission">
-      <actuator name="right_arm_a3" />
+    <transmission name="right_arm_t3">
+      <type>transmission_interface/SimpleTransmission</type>
       <joint name="right_arm_j3" />
-      <mechanicalReduction>1.0</mechanicalReduction>
+      <actuator name="right_arm_a3">
+        <hardwareInterface>PositionJointInterface</hardwareInterface>
+        <mechanicalReduction>1.0</mechanicalReduction>
+      </actuator>
     </transmission>
     <!-- Elbow flex -->
-    <transmission name="right_arm_t4" type="pr2_mechanism_model/SimpleTransmission">
-      <actuator name="right_arm_a4" />
+    <transmission name="right_arm_t4">
+      <type>transmission_interface/SimpleTransmission</type>
       <joint name="right_arm_j4" />
-      <mechanicalReduction>1.0</mechanicalReduction>
+      <actuator name="right_arm_a4">
+        <hardwareInterface>PositionJointInterface</hardwareInterface>
+        <mechanicalReduction>1.0</mechanicalReduction>
+      </actuator>
     </transmission>
   </macro>
   <!-- ============================   Forearm   ============================ -->
   <macro name="m3_r_forearm_transmission" params="side parent reflect">
-    <transmission name="right_arm_t5" type="pr2_mechanism_model/SimpleTransmission">
-      <actuator name="right_arm_a5" />
+    <transmission name="right_arm_t5">
+      <type>transmission_interface/SimpleTransmission</type>
       <joint name="right_arm_j5" />
-      <mechanicalReduction>1.0</mechanicalReduction>
+      <actuator name="right_arm_a5">
+        <hardwareInterface>PositionJointInterface</hardwareInterface>
+        <mechanicalReduction>1.0</mechanicalReduction>
+      </actuator>
     </transmission>
     <!-- Wrist flex -->
-    <transmission name="right_arm_t6" type="pr2_mechanism_model/SimpleTransmission">
-      <actuator name="right_arm_a6" />
+    <transmission name="right_arm_t6">
+      <type>transmission_interface/SimpleTransmission</type>
       <joint name="right_arm_j6" />
-      <mechanicalReduction>1.0</mechanicalReduction>
+      <actuator name="right_arm_a6">
+        <hardwareInterface>PositionJointInterface</hardwareInterface>
+        <mechanicalReduction>1.0</mechanicalReduction>
+      </actuator>
     </transmission>
   </macro>

File: gt_meka_description/urdf/transmissions_hydro/SIMC_head_defs.transmission.xacro (robot description, xacro)
@@ -5,42 +5,73 @@
   <property name="M_PI" value="3.1415926535897931" />
   <macro name="m3_neck_transmission">
-  <transmission name="head_t0" type="pr2_mechanism_model/SimpleTransmission">
-      <actuator name="head_a0"/>
-      <joint name="head_j0"/>
-    <mechanicalReduction>1</mechanicalReduction>
-  </transmission>
-  <transmission name="head_t1" type="pr2_mechanism_model/SimpleTransmission">
-      <actuator name="head_a1"/>
-      <joint name="head_j1"/>
-    <mechanicalReduction>1</mechanicalReduction>
-  </transmission>
-  <transmission name="head_t2" type="pr2_mechanism_model/SimpleTransmission">
-      <actuator name="head_a2"/>
-      <joint name="head_j2"/>
-    <mechanicalReduction>1</mechanicalReduction>
-  </transmission>
-  <transmission name="head_t3" type="pr2_mechanism_model/SimpleTransmission">
-      <actuator name="head_a3"/>
-      <joint name="head_j3"/>
-    <mechanicalReduction>1</mechanicalReduction>
-  </transmission>
+    <transmission name="head_t0">
+      <type>transmission_interface/SimpleTransmission</type>
+      <joint name="head_j0" />
+      <actuator name="head_a0">
+        <hardwareInterface>PositionJointInterface</hardwareInterface>
+        <mechanicalReduction>1.0</mechanicalReduction>
+      </actuator>
+    </transmission>
+    <transmission name="head_t1">
+      <type>transmission_interface/SimpleTransmission</type>
+      <joint name="head_j1" />
+      <actuator name="head_a1">
+        <hardwareInterface>PositionJointInterface</hardwareInterface>
+        <mechanicalReduction>1.0</mechanicalReduction>
+      </actuator>
+    </transmission>
+    <transmission name="head_t2">
+      <type>transmission_interface/SimpleTransmission</type>
+      <joint name="head_j2" />
+      <actuator name="head_a2">
+        <hardwareInterface>PositionJointInterface</hardwareInterface>
+        <mechanicalReduction>1.0</mechanicalReduction>
+      </actuator>
+    </transmission>
+    <transmission name="head_t3">
+      <type>transmission_interface/SimpleTransmission</type>
+      <joint name="head_j3" />
+      <actuator name="head_a3">
+        <hardwareInterface>PositionJointInterface</hardwareInterface>
+        <mechanicalReduction>1.0</mechanicalReduction>
+      </actuator>
+    </transmission>
 </macro>
+  <!-- Not using eye or ears right now - so incorrect -->
   <macro name="m3_eye_transmission">
-  <transmission name="head_t4" type="pr2_mechanism_model/SimpleTransmission">
-      <actuator name="head_a4"/>
-      <joint name="head_j4"/>
-    <mechanicalReduction>1</mechanicalReduction>
-  </transmission>
-  <transmission name="head_t5" type="pr2_mechanism_model/SimpleTransmission">
-      <actuator name="head_a5"/>
-      <joint name="head_j5"/>
-    <mechanicalReduction>1</mechanicalReduction>
-  </transmission>
-  <transmission name="head_t6" type="pr2_mechanism_model/SimpleTransmission">
-      <actuator name="head_a6"/>
-      <joint name="head_j6"/>
-    <mechanicalReduction>1</mechanicalReduction>
-  </transmission>
-  <transmission name="head_t7_rt_eyelid_top" type="pr2_mechanism_model/SimpleTransmission">
+    <transmission name="head_t4">
+      <type>transmission_interface/SimpleTransmission</type>
+      <joint name="head_j4" />
+      <actuator name="head_a4">
+        <hardwareInterface>PositionJointInterface</hardwareInterface>
+        <mechanicalReduction>1.0</mechanicalReduction>
+      </actuator>
+    </transmission>
+    <transmission name="head_t5">
+      <type>transmission_interface/SimpleTransmission</type>
+      <joint name="head_j5" />
+      <actuator name="head_a5">
+        <hardwareInterface>PositionJointInterface</hardwareInterface>
+        <mechanicalReduction>1.0</mechanicalReduction>
+      </actuator>
+    </transmission>
+    <transmission name="head_t6">
+      <type>transmission_interface/SimpleTransmission</type>
+      <joint name="head_j6" />
+      <actuator name="head_a6">
+        <hardwareInterface>PositionJointInterface</hardwareInterface>
+        <mechanicalReduction>1.0</mechanicalReduction>
+      </actuator>
+    </transmission>
+    <transmission name="head_t7">
+      <type>transmission_interface/SimpleTransmission</type>
+      <joint name="head_j7" />
+      <actuator name="head_a7">
+        <hardwareInterface>PositionJointInterface</hardwareInterface>
+        <mechanicalReduction>1.0</mechanicalReduction>
+      </actuator>
+    </transmission>
+  <!-- Correct/Old names for when we actually control the eyelids -->
+  <!--transmission name="head_t7_rt_eyelid_top" type="pr2_mechanism_model/SimpleTransmission">
       <actuator name="head_a7_rt_eyelid_top"/>
       <joint name="head_j7_rt_eyelid_top"/>
@@ -61,32 +92,44 @@
       <joint name="head_j7_lt_eyelid_bottom"/>
     <mechanicalReduction>1</mechanicalReduction>
-  </transmission>
+  </transmission-->
 </macro>
   <macro name="m3_ear_transmission">
-  <transmission name="head_t8" type="pr2_mechanism_model/SimpleTransmission">
-      <actuator name="head_a8"/>
-      <joint name="head_j8"/>
-    <mechanicalReduction>1</mechanicalReduction>
-  </transmission>
-  <transmission name="head_t9" type="pr2_mechanism_model/SimpleTransmission">
-      <actuator name="head_a9"/>
-      <joint name="head_j9"/>
-    <mechanicalReduction>1</mechanicalReduction>
-  </transmission>
-  <transmission name="head_t10" type="pr2_mechanism_model/SimpleTransmission">
-      <actuator name="head_a10"/>
-      <joint name="head_j10"/>
-    <mechanicalReduction>1</mechanicalReduction>
-  </transmission>
-  <transmission name="head_t11" type="pr2_mechanism_model/SimpleTransmission">
-      <actuator name="head_a11"/>
-      <joint name="head_j11"/>
-    <mechanicalReduction>1</mechanicalReduction>
-  </transmission>
+    <transmission name="head_t8">
+      <type>transmission_interface/SimpleTransmission</type>
+      <joint name="head_j8" />
+      <actuator name="head_a8">
+        <hardwareInterface>PositionJointInterface</hardwareInterface>
+        <mechanicalReduction>1.0</mechanicalReduction>
+      </actuator>
+    </transmission>
+    <transmission name="head_t9">
+      <type>transmission_interface/SimpleTransmission</type>
+      <joint name="head_j9" />
+      <actuator name="head_a9">
+        <hardwareInterface>PositionJointInterface</hardwareInterface>
+        <mechanicalReduction>1.0</mechanicalReduction>
+      </actuator>
+    </transmission>
+    <transmission name="head_t10">
+      <type>transmission_interface/SimpleTransmission</type>
+      <joint name="head_j10" />
+      <actuator name="head_a10">
+        <hardwareInterface>PositionJointInterface</hardwareInterface>
+        <mechanicalReduction>1.0</mechanicalReduction>
+      </actuator>
+    </transmission>
+    <transmission name="head_t11">
+      <type>transmission_interface/SimpleTransmission</type>
+      <joint name="head_j11" />
+      <actuator name="head_a11">
+        <hardwareInterface>PositionJointInterface</hardwareInterface>
+        <mechanicalReduction>1.0</mechanicalReduction>
+      </actuator>
+    </transmission>
 </macro>
   <macro name="m3_head_transmission">
     <m3_neck_transmission/>
-    <!--m3_eye_transmission/>
-    <m3_ear_transmission/-->
+    <m3_eye_transmission/>
+    <m3_ear_transmission/>
   </macro>
 </robot>

File: gt_meka_description/urdf/transmissions_hydro/zlift_defs.transmission.xacro (robot description, xacro)
@@ -6,5 +6,5 @@
       <joint name="${name}_joint" />
       <actuator name="${name}_a0">
-        <hardwareInterface>EffortJointInterface</hardwareInterface>
+        <hardwareInterface>PositionJointInterface</hardwareInterface>
         <mechanicalReduction>1</mechanicalReduction>
       </actuator>
