Commit message: updated joint limits for the right hand and lower pid values for gazebo

File: gt_meka_description/urdf/H2R4_r_hand_defs.urdf.xacro (robot description, xacro)
@@ -83,5 +83,6 @@
     <joint name="right_hand_j1" type="revolute">
       <axis xyz="0 -1 0"/>
-     <limit effort="100" velocity="${75*M_PI/180}" lower="${-80.919*M_PI/180}" upper="${80.91*M_PI/180}" />
+      <!--limit effort="100" velocity="${75*M_PI/180}" lower="${-80.919*M_PI/180}" upper="${80.91*M_PI/180}" /-->
+	  <limit effort="100" velocity="${50*M_PI/180}" lower="${-7.072*M_PI/180}" upper="${90.0*M_PI/180}" />
       <origin xyz="-0.018 0 0" rpy="0 0 0" />
       <parent link="thumb0"/>
@@ -117,5 +118,6 @@
       <parent link="thumb1" />
       <child link="thumb2"/>
-      <limit effort="100" velocity="${50*M_PI/180}" lower="${-14.94*M_PI/180}" upper="${14.94*M_PI/180}" />
+      <!--limit effort="100" velocity="${50*M_PI/180}" lower="${-14.94*M_PI/180}" upper="${14.94*M_PI/180}" /-->
+	  <limit effort="100" velocity="${50*M_PI/180}" lower="${-7.072*M_PI/180}" upper="${90.0*M_PI/180}" />
     </joint>
     <link name="thumb2">
@@ -149,5 +151,6 @@
       <parent link="palm" />
       <child link="index0"/>
-	<limit effort="100" velocity="${50*M_PI/180}" lower="${-7.072*M_PI/180}" upper="${37.072*M_PI/180}" />
+	<!--limit effort="100" velocity="${50*M_PI/180}" lower="${-7.072*M_PI/180}" upper="${37.072*M_PI/180}" /-->
+	<limit effort="100" velocity="${50*M_PI/180}" lower="${-7.072*M_PI/180}" upper="${90.0*M_PI/180}" />
     </joint>
     <link name="index0">
@@ -177,5 +180,6 @@
     <joint name="right_hand_j4" type="revolute">
       <axis xyz="0 1 0" />
-      <limit effort="100" velocity="${1600*M_PI/180}" lower="${-34.99*M_PI/180}" upper="${34.99*M_PI/180}" />
+      <!--limit effort="100" velocity="${1600*M_PI/180}" lower="${-34.99*M_PI/180}" upper="${34.99*M_PI/180}" /-->
+	  <limit effort="100" velocity="${50*M_PI/180}" lower="${-7.072*M_PI/180}" upper="${90.0*M_PI/180}" />
       <origin xyz="0 0 -0.044" rpy="0 0 0" />
       <parent link="index0"/>
@@ -208,5 +212,6 @@
     <joint name="right_hand_j5" type="revolute">
       <axis xyz="0 1 0" />
-      <limit effort="100" velocity="${1600*M_PI/180}" lower="${-34.21*M_PI/180}" upper="${34.213*M_PI/180}" />
+      <!--limit effort="100" velocity="${1600*M_PI/180}" lower="${-34.21*M_PI/180}" upper="${34.213*M_PI/180}" /-->
+	  <limit effort="100" velocity="${50*M_PI/180}" lower="${-7.072*M_PI/180}" upper="${90.0*M_PI/180}" />
       <origin xyz="0 0 -0.032" rpy="0 0 0" />
       <parent link="index1"/>
@@ -243,5 +248,6 @@
       <parent link="palm" />
       <child link="ring0"/>
-	<limit effort="100" velocity="${50*M_PI/180}" lower="${-7.072*M_PI/180}" upper="${37.072*M_PI/180}" />
+	  <!--limit effort="100" velocity="${50*M_PI/180}" lower="${-7.072*M_PI/180}" upper="${37.072*M_PI/180}" /-->
+	  <limit effort="100" velocity="${50*M_PI/180}" lower="${-7.072*M_PI/180}" upper="${90.0*M_PI/180}" />
     </joint>
     <link name="ring0">
@@ -271,5 +277,6 @@
     <joint name="right_hand_j7" type="revolute">
       <axis xyz="0 1 0" />
-      <limit effort="100" velocity="${1600*M_PI/180}" lower="${-34.99*M_PI/180}" upper="${34.99*M_PI/180}" />
+      <!--limit effort="100" velocity="${1600*M_PI/180}" lower="${-34.99*M_PI/180}" upper="${34.99*M_PI/180}" /-->
+	  <limit effort="100" velocity="${50*M_PI/180}" lower="${-7.072*M_PI/180}" upper="${90.0*M_PI/180}" />
       <origin xyz="0 0 -0.044" rpy="0 0 0" />
       <parent link="ring0"/>
@@ -302,5 +309,6 @@
     <joint name="right_hand_j8" type="revolute">
       <axis xyz="0 1 0" />
-      <limit effort="100" velocity="${1600*M_PI/180}" lower="${-34.21*M_PI/180}" upper="${34.213*M_PI/180}" />
+      <!--limit effort="100" velocity="${1600*M_PI/180}" lower="${-34.21*M_PI/180}" upper="${34.213*M_PI/180}" /-->
+	  <limit effort="100" velocity="${50*M_PI/180}" lower="${-7.072*M_PI/180}" upper="${90.0*M_PI/180}" />
       <origin xyz="0 0 -0.032" rpy="0 0 0" />
       <parent link="ring1"/>
@@ -337,5 +345,6 @@
       <parent link="palm" />
       <child link="pinky0"/>
-	<limit effort="100" velocity="${50*M_PI/180}" lower="${-7.072*M_PI/180}" upper="${37.072*M_PI/180}" />
+	  <!--limit effort="100" velocity="${50*M_PI/180}" lower="${-7.072*M_PI/180}" upper="${37.072*M_PI/180}" /-->
+	  <limit effort="100" velocity="${50*M_PI/180}" lower="${-7.072*M_PI/180}" upper="${90.0*M_PI/180}" />
     </joint>
     <link name="pinky0">
@@ -365,5 +374,6 @@
     <joint name="right_hand_j10" type="revolute">
       <axis xyz="0 1 0" />
-      <limit effort="100" velocity="${1600*M_PI/180}" lower="${-34.99*M_PI/180}" upper="${34.99*M_PI/180}" />
+      <!--limit effort="100" velocity="${1600*M_PI/180}" lower="${-34.99*M_PI/180}" upper="${34.99*M_PI/180}" /-->
+	  <limit effort="100" velocity="${50*M_PI/180}" lower="${-7.072*M_PI/180}" upper="${90.0*M_PI/180}" />
       <origin xyz="0 0 -0.044" rpy="0 0 0" />
       <parent link="pinky0"/>
@@ -396,5 +406,6 @@
     <joint name="right_hand_j11" type="revolute">
       <axis xyz="0 1 0" />
-      <limit effort="100" velocity="${1600*M_PI/180}" lower="${-34.21*M_PI/180}" upper="${34.213*M_PI/180}" />
+      <!--limit effort="100" velocity="${1600*M_PI/180}" lower="${-34.21*M_PI/180}" upper="${34.213*M_PI/180}" /-->
+	  <limit effort="100" velocity="${50*M_PI/180}" lower="${-7.072*M_PI/180}" upper="${90.0*M_PI/180}" />
       <origin xyz="0 0 -0.032" rpy="0 0 0" />
       <parent link="pinky1"/>
