Commit message: added in support for curi's hand

File: gt_meka_description/urdf/H2R4_l_hand_defs.urdf.xacro (robot description, xacro)
@@ -47,5 +47,5 @@
     <joint name="left_hand_j0" type="revolute">
       <axis xyz="0 0 -1" />
-      <origin xyz="-0.02 -0.028 -0.03" rpy="0 0 0" />
+      <origin xyz="-0.02 -0.028 -0.03" rpy="0 0 1.57" />
       <parent link="l_palm"/>
       <child link="l_thumb0"/>

File: gt_meka_description/urdf/simco-groovy.urdf.xacro (robot description, xacro)
@@ -30,4 +30,6 @@
   <include filename="./transmissions/zlift_defs.transmission.xacro" />
   <include filename="./transmissions/SIMC_head_defs.transmission.xacro" />
+  <include filename="./transmissions/H2R4_r_hand_defs.transmission.xacro" />
+  <include filename="./transmissions/H2R4_l_hand_defs.transmission.xacro" />
   <link name="world" />
   <meka_base reflect="1" parent="world">
@@ -35,5 +37,6 @@
   </meka_base>
   <meka_zlift  side="r" reflect="1" parent="dummy_3">
-    <origin xyz="0.42 0.0 0.6137" rpy="0 0 0" />
+    <!--origin xyz="0.42 0.0 0.6137" rpy="0 0 0" /-->
+    <origin xyz="0.42 0.0 0.85" rpy="0 0 0" />
   </meka_zlift>
   <!-- Torso -->
@@ -75,12 +78,10 @@
   </m3_l_arm>
   <!-- Add Hands -->
-  <!--
   <m3_r_hand side="r" reflect="1" parent="handmount_RIGHT">
     <origin xyz="0.0 0.0 0.0" rpy="0 0 0" />
   </m3_r_hand>
-  <m3_l_hand side="l" reflect="1" parent="handmount_LEFT">
+  <m3_l_hand side="l" reflect="-1" parent="handmount_LEFT">
     <origin xyz="0.0 0.0 0.0" rpy="0 0 0" />
   </m3_l_hand>
-  -->
   <!-- Add Head -->
   <m3_head side="r" reflect="1" parent="chest_link">
@@ -92,3 +93,5 @@
   <m3_l_arm_transmission side="l" reflect="1" parent="torso_lift_link"/>
   <m3_head_transmission />
+  <m3_r_hand_transmission />
+  <m3_l_hand_transmission />
 </robot>

Commit message: semi working inertia values for both hands

File: gt_meka_description/urdf/H2R4_l_hand_defs.urdf.xacro (robot description, xacro)
@@ -55,8 +55,8 @@
       <inertial>
         <mass value="0.0117" />
-	<origin xyz="0.0 0.0 0.0"/>
-	<inertia ixx="0.0"
-	iyy="0.0"
-	izz="0.0"
+	<origin xyz="-0.007 -0.00007 -0.0018"/>
+	<inertia ixx="0.00011"
+	iyy="0.00014"
+	izz="0.0008"
 	ixy="0.0"
 	ixz="0.0"
@@ -86,8 +86,8 @@
       <inertial>
         <mass value="0.0344" />
-	<origin xyz="0.0 0.0 0.0"/>
-	<inertia ixx="0.0"
-	iyy="0.0"
-	izz="0.0"
+	<origin xyz="-0.0015 -0.000014 -0.000081"/>
+	<inertia ixx="0.001"
+	iyy="0.004"
+	izz="0.004"
 	ixy="0.0"
 	ixz="0.0"
@@ -117,8 +117,8 @@
       <inertial>
         <mass value="0.01" />
-	<origin xyz="0.0 0.0 0.0"/>
-	<inertia ixx="0.0"
-	iyy="0.0"
-	izz="0.0"
+	<origin xyz="-0.0009 -0.0003 0.0006"/>
+	<inertia ixx="0.001"
+	iyy="0.004"
+	izz="0.004"
 	ixy="0.0"
 	ixz="0.0"
@@ -149,8 +149,8 @@
       <inertial>
         <mass value="0.01" />
-	<origin xyz="0.0 0.0 0.0"/>
-	<inertia ixx="0.0"
-	iyy="0.0"
-	izz="0.0"
+	<origin xyz="-0.000416 -0.000061 -0.0012"/>
+	<inertia ixx="0.03"
+	iyy="0.03"
+	izz="0.08"
 	ixy="0.0"
 	ixz="0.0"
@@ -180,8 +180,8 @@
       <inertial>
         <mass value="0.0429" />
-	<origin xyz="0.0 0.0 0.0"/>
-	<inertia ixx="0.0"
-	iyy="0.0"
-	izz="0.0"
+	<origin xyz="0.003 0.0018 -0.08"/>
+	<inertia ixx="0.01"
+	iyy="0.01"
+	izz="0.003"
 	ixy="0.0"
 	ixz="0.0"
@@ -211,8 +211,8 @@
       <inertial>
         <mass value="0.01" />
-	<origin xyz="0.0 0.0 0.0"/>
-	<inertia ixx="0.0"
-	iyy="0.0"
-	izz="0.0"
+	<origin xyz="0.006 -0.006 -0.002"/>
+	<inertia ixx="0.04"
+	iyy="0.04"
+	izz="0.001"
 	ixy="0.0"
 	ixz="0.0"
@@ -243,8 +243,8 @@
       <inertial>
         <mass value="0.01" />
-	<origin xyz="0.0 0.0 0.0"/>
-	<inertia ixx="0.0"
-	iyy="0.0"
-	izz="0.0"
+	<origin xyz="-0.000416 -0.000061 -0.0012"/>
+	<inertia ixx="0.03"
+	iyy="0.03"
+	izz="0.08"
 	ixy="0.0"
 	ixz="0.0"
@@ -274,8 +274,8 @@
       <inertial>
         <mass value="0.0429" />
-	<origin xyz="0.0 0.0 0.0"/>
-	<inertia ixx="0.0"
-	iyy="0.0"
-	izz="0.0"
+	<origin xyz="0.003 0.0018 -0.08"/>
+	<inertia ixx="0.01"
+	iyy="0.01"
+	izz="0.003"
 	ixy="0.0"
 	ixz="0.0"
@@ -305,8 +305,8 @@
       <inertial>
         <mass value="0.01" />
-	<origin xyz="0.0 0.0 0.0"/>
-	<inertia ixx="0.0"
-	iyy="0.0"
-	izz="0.0"
+	<origin xyz="0.006 -0.006 -0.002"/>
+	<inertia ixx="0.04"
+	iyy="0.04"
+	izz="0.001"
 	ixy="0.0"
 	ixz="0.0"
@@ -337,8 +337,8 @@
       <inertial>
         <mass value="0.01" />
-	<origin xyz="0.0 0.0 0.0"/>
-	<inertia ixx="0.0"
-	iyy="0.0"
-	izz="0.0"
+	<origin xyz="-0.000416 -0.000061 -0.0012"/>
+	<inertia ixx="0.03"
+	iyy="0.03"
+	izz="0.08"
 	ixy="0.0"
 	ixz="0.0"
@@ -368,8 +368,8 @@
       <inertial>
         <mass value="0.0429" />
-	<origin xyz="0.0 0.0 0.0"/>
-	<inertia ixx="0.0"
-	iyy="0.0"
-	izz="0.0"
+	<origin xyz="0.003 0.0018 -0.08"/>
+	<inertia ixx="0.01"
+	iyy="0.01"
+	izz="0.003"
 	ixy="0.0"
 	ixz="0.0"
@@ -399,8 +399,8 @@
       <inertial>
         <mass value="0.01" />
-	<origin xyz="0.0 0.0 0.0"/>
-	<inertia ixx="0.0"
-	iyy="0.0"
-	izz="0.0"
+	<origin xyz="0.006 -0.006 -0.002"/>
+	<inertia ixx="0.04"
+	iyy="0.04"
+	izz="0.001"
 	ixy="0.0"
 	ixz="0.0"

File: gt_meka_description/urdf/H2R4_r_hand_defs.urdf.xacro (robot description, xacro)
@@ -49,4 +49,5 @@
     </link>
 <!-- Start Thumb -->
+  <!-- thumb inertia might be off because of direct copy from left hand -->
     <joint name="right_hand_j0" type="revolute">
       <axis xyz="0 0 1" />
@@ -59,11 +60,11 @@
       <inertial>
         <mass value="0.0117" />
-	<origin xyz="0.0 0.0 0.0"/>
-	<inertia ixx="0.0"
-	iyy="0.0"
-	izz="0.0"
-	ixy="0.0"
-	ixz="0.0"
-	iyz="0.0" />
+    <origin xyz="-0.007 -0.00007 -0.0018"/>
+    <inertia ixx="0.00011"
+    iyy="0.00014"
+    izz="0.0008"
+    ixy="0.0"
+    ixz="0.0"
+    iyz="0.0" />
       </inertial>
       <visual>
@@ -90,11 +91,11 @@
       <inertial>
         <mass value="0.0344" />
-	<origin xyz="0.0 0.0 0.0"/>
-	<inertia ixx="0.0"
-	iyy="0.0"
-	izz="0.0"
-	ixy="0.0"
-	ixz="0.0"
-	iyz="0.0" />
+    <origin xyz="-0.0015 -0.000014 -0.000081"/>
+    <inertia ixx="0.001"
+    iyy="0.004"
+    izz="0.004"
+    ixy="0.0"
+    ixz="0.0"
+    iyz="0.0" />
       </inertial>
       <visual>
@@ -121,11 +122,11 @@
       <inertial>
         <mass value="0.01" />
-	<origin xyz="0.0 0.0 0.0"/>
-	<inertia ixx="0.0"
-	iyy="0.0"
-	izz="0.0"
-	ixy="0.0"
-	ixz="0.0"
-	iyz="0.0" />
+    <origin xyz="-0.0009 -0.0003 0.0006"/>
+    <inertia ixx="0.001"
+    iyy="0.004"
+    izz="0.004"
+    ixy="0.0"
+    ixz="0.0"
+    iyz="0.0" />
       </inertial>
       <visual>
@@ -153,11 +154,11 @@
       <inertial>
         <mass value="0.01" />
-	<origin xyz="0.0 0.0 0.0"/>
-	<inertia ixx="0.0"
-	iyy="0.0"
-	izz="0.0"
-	ixy="0.0"
-	ixz="0.0"
-	iyz="0.0" />
+    <origin xyz="-0.000416 -0.000061 -0.0012"/>
+    <inertia ixx="0.03"
+    iyy="0.03"
+    izz="0.08"
+    ixy="0.0"
+    ixz="0.0"
+    iyz="0.0" />
       </inertial>
       <visual>
@@ -184,11 +185,11 @@
       <inertial>
         <mass value="0.0429" />
-	<origin xyz="0.0 0.0 0.0"/>
-	<inertia ixx="0.0"
-	iyy="0.0"
-	izz="0.0"
-	ixy="0.0"
-	ixz="0.0"
-	iyz="0.0" />
+    <origin xyz="0.003 0.0018 -0.08"/>
+    <inertia ixx="0.01"
+    iyy="0.01"
+    izz="0.003"
+    ixy="0.0"
+    ixz="0.0"
+    iyz="0.0" />
       </inertial>
       <visual>
@@ -215,11 +216,11 @@
       <inertial>
         <mass value="0.01" />
-	<origin xyz="0.0 0.0 0.0"/>
-	<inertia ixx="0.0"
-	iyy="0.0"
-	izz="0.0"
-	ixy="0.0"
-	ixz="0.0"
-	iyz="0.0" />
+    <origin xyz="0.006 -0.006 -0.002"/>
+    <inertia ixx="0.04"
+    iyy="0.04"
+    izz="0.001"
+    ixy="0.0"
+    ixz="0.0"
+    iyz="0.0" />
       </inertial>
       <visual>
@@ -247,11 +248,11 @@
       <inertial>
         <mass value="0.01" />
-	<origin xyz="0.0 0.0 0.0"/>
-	<inertia ixx="0.0"
-	iyy="0.0"
-	izz="0.0"
-	ixy="0.0"
-	ixz="0.0"
-	iyz="0.0" />
+    <origin xyz="-0.000416 -0.000061 -0.0012"/>
+    <inertia ixx="0.03"
+    iyy="0.03"
+    izz="0.08"
+    ixy="0.0"
+    ixz="0.0"
+    iyz="0.0" />
       </inertial>
       <visual>
@@ -278,11 +279,11 @@
       <inertial>
         <mass value="0.0429" />
-	<origin xyz="0.0 0.0 0.0"/>
-	<inertia ixx="0.0"
-	iyy="0.0"
-	izz="0.0"
-	ixy="0.0"
-	ixz="0.0"
-	iyz="0.0" />
+    <origin xyz="0.003 0.0018 -0.08"/>
+    <inertia ixx="0.01"
+    iyy="0.01"
+    izz="0.003"
+    ixy="0.0"
+    ixz="0.0"
+    iyz="0.0" />
       </inertial>
       <visual>
@@ -309,11 +310,11 @@
       <inertial>
         <mass value="0.01" />
-	<origin xyz="0.0 0.0 0.0"/>
-	<inertia ixx="0.0"
-	iyy="0.0"
-	izz="0.0"
-	ixy="0.0"
-	ixz="0.0"
-	iyz="0.0" />
+    <origin xyz="0.006 -0.006 -0.002"/>
+    <inertia ixx="0.04"
+    iyy="0.04"
+    izz="0.001"
+    ixy="0.0"
+    ixz="0.0"
+    iyz="0.0" />
       </inertial>
       <visual>
@@ -341,11 +342,11 @@
       <inertial>
         <mass value="0.01" />
-	<origin xyz="0.0 0.0 0.0"/>
-	<inertia ixx="0.0"
-	iyy="0.0"
-	izz="0.0"
-	ixy="0.0"
-	ixz="0.0"
-	iyz="0.0" />
+    <origin xyz="-0.000416 -0.000061 -0.0012"/>
+    <inertia ixx="0.03"
+    iyy="0.03"
+    izz="0.08"
+    ixy="0.0"
+    ixz="0.0"
+    iyz="0.0" />
       </inertial>
       <visual>
@@ -372,11 +373,11 @@
       <inertial>
         <mass value="0.0429" />
-	<origin xyz="0.0 0.0 0.0"/>
-	<inertia ixx="0.0"
-	iyy="0.0"
-	izz="0.0"
-	ixy="0.0"
-	ixz="0.0"
-	iyz="0.0" />
+    <origin xyz="0.003 0.0018 -0.08"/>
+    <inertia ixx="0.01"
+    iyy="0.01"
+    izz="0.003"
+    ixy="0.0"
+    ixz="0.0"
+    iyz="0.0" />
       </inertial>
       <visual>
@@ -403,11 +404,11 @@
       <inertial>
         <mass value="0.01" />
-	<origin xyz="0.0 0.0 0.0"/>
-	<inertia ixx="0.0"
-	iyy="0.0"
-	izz="0.0"
-	ixy="0.0"
-	ixz="0.0"
-	iyz="0.0" />
+    <origin xyz="0.006 -0.006 -0.002"/>
+    <inertia ixx="0.04"
+    iyy="0.04"
+    izz="0.001"
+    ixy="0.0"
+    ixz="0.0"
+    iyz="0.0" />
       </inertial>
       <visual>

Commit message: fixed timing issue using queues, also added in support for left hand

File: gt_meka_description/urdf/H2R4_l_hand_defs.urdf.xacro (robot description, xacro)
@@ -50,5 +50,6 @@
       <parent link="l_palm"/>
       <child link="l_thumb0"/>
-      <limit effort="100" velocity="${20.0*M_PI/180}" lower="${-40*M_PI/180}" upper="${15*M_PI/180}" />
+      <!--limit effort="100" velocity="${20.0*M_PI/180}" lower="${-40*M_PI/180}" upper="${15*M_PI/180}" /-->
+	  <limit effort="100" velocity="${40.0*M_PI/180}" lower="${-7.072*M_PI/180}" upper="${90.0*M_PI/180}" />
     </joint>
     <link name="l_thumb0">
@@ -78,5 +79,6 @@
     <joint name="left_hand_j1" type="revolute">
       <axis xyz="0 -1 0"/>
-     <limit effort="100" velocity="${75*M_PI/180}" lower="${-80.919*M_PI/180}" upper="${80.91*M_PI/180}" />
+     <!--limit effort="100" velocity="${75*M_PI/180}" lower="${-80.919*M_PI/180}" upper="${80.91*M_PI/180}" /-->
+	  <limit effort="100" velocity="${75.0*M_PI/180}" lower="${-7.072*M_PI/180}" upper="${90.0*M_PI/180}" />
       <origin xyz="-0.018 0 0" rpy="0 0 0" />
       <parent link="l_thumb0"/>
@@ -112,5 +114,6 @@
       <parent link="l_thumb1" />
       <child link="l_thumb2"/>
-      <limit effort="100" velocity="${50*M_PI/180}" lower="${-14.94*M_PI/180}" upper="${14.94*M_PI/180}" />
+      <!--limit effort="100" velocity="${50*M_PI/180}" lower="${-14.94*M_PI/180}" upper="${14.94*M_PI/180}" /-->
+	  <limit effort="100" velocity="${50.0*M_PI/180}" lower="${-7.072*M_PI/180}" upper="${90.0*M_PI/180}" />
     </joint>
     <link name="l_thumb2">
@@ -144,5 +147,6 @@
       <parent link="l_palm" />
       <child link="l_index0"/>
-	<limit effort="100" velocity="${50*M_PI/180}" lower="${-7.072*M_PI/180}" upper="${37.072*M_PI/180}" />
+	<!--limit effort="100" velocity="${50*M_PI/180}" lower="${-7.072*M_PI/180}" upper="${37.072*M_PI/180}" /-->
+	<limit effort="100" velocity="${50*M_PI/180}" lower="${-7.072*M_PI/180}" upper="${90.0*M_PI/180}" />
     </joint>
     <link name="l_index0">
@@ -172,5 +176,6 @@
     <joint name="left_hand_j4" type="revolute">
       <axis xyz="0 1 0" />
-      <limit effort="100" velocity="${1600*M_PI/180}" lower="${-34.99*M_PI/180}" upper="${34.99*M_PI/180}" />
+      <!--limit effort="100" velocity="${1600*M_PI/180}" lower="${-34.99*M_PI/180}" upper="${34.99*M_PI/180}" /-->
+	  <limit effort="100" velocity="${1600*M_PI/180}" lower="${-7.072*M_PI/180}" upper="${90.0*M_PI/180}" />
       <origin xyz="0 0 -0.044" rpy="0 0 0" />
       <parent link="l_index0"/>
@@ -203,5 +208,6 @@
     <joint name="left_hand_j5" type="revolute">
       <axis xyz="0 1 0" />
-      <limit effort="100" velocity="${1600*M_PI/180}" lower="${-34.21*M_PI/180}" upper="${34.213*M_PI/180}" />
+      <!--limit effort="100" velocity="${1600*M_PI/180}" lower="${-34.21*M_PI/180}" upper="${34.213*M_PI/180}" /-->
+	  <limit effort="100" velocity="${1600*M_PI/180}" lower="${-7.072*M_PI/180}" upper="${90.0*M_PI/180}" />
       <origin xyz="0 0 -0.032" rpy="0 0 0" />
       <parent link="l_index1"/>
@@ -238,5 +244,6 @@
       <parent link="l_palm" />
       <child link="l_ring0"/>
-	<limit effort="100" velocity="${50*M_PI/180}" lower="${-7.072*M_PI/180}" upper="${37.072*M_PI/180}" />
+	  <!--limit effort="100" velocity="${50*M_PI/180}" lower="${-7.072*M_PI/180}" upper="${37.072*M_PI/180}" /-->
+	  <limit effort="100" velocity="${1600*M_PI/180}" lower="${-7.072*M_PI/180}" upper="${90.0*M_PI/180}" />
     </joint>
     <link name="l_ring0">
@@ -266,5 +273,6 @@
     <joint name="left_hand_j7" type="revolute">
       <axis xyz="0 1 0" />
-      <limit effort="100" velocity="${1600*M_PI/180}" lower="${-34.99*M_PI/180}" upper="${34.99*M_PI/180}" />
+      <!--limit effort="100" velocity="${1600*M_PI/180}" lower="${-34.99*M_PI/180}" upper="${34.99*M_PI/180}" /-->
+	  <limit effort="100" velocity="${1600*M_PI/180}" lower="${-7.072*M_PI/180}" upper="${90.0*M_PI/180}" />
       <origin xyz="0 0 -0.044" rpy="0 0 0" />
       <parent link="l_ring0"/>
@@ -297,5 +305,6 @@
     <joint name="left_hand_j8" type="revolute">
       <axis xyz="0 1 0" />
-      <limit effort="100" velocity="${1600*M_PI/180}" lower="${-34.21*M_PI/180}" upper="${34.213*M_PI/180}" />
+      <!--limit effort="100" velocity="${1600*M_PI/180}" lower="${-34.21*M_PI/180}" upper="${34.213*M_PI/180}" /-->
+	  <limit effort="100" velocity="${1600*M_PI/180}" lower="${-7.072*M_PI/180}" upper="${90.0*M_PI/180}" />
       <origin xyz="0 0 -0.032" rpy="0 0 0" />
       <parent link="l_ring1"/>
@@ -332,5 +341,6 @@
       <parent link="l_palm" />
       <child link="l_pinky0"/>
-	<limit effort="100" velocity="${50*M_PI/180}" lower="${-7.072*M_PI/180}" upper="${37.072*M_PI/180}" />
+	  <!--limit effort="100" velocity="${50*M_PI/180}" lower="${-7.072*M_PI/180}" upper="${37.072*M_PI/180}" /-->
+	  <limit effort="100" velocity="${1600*M_PI/180}" lower="${-7.072*M_PI/180}" upper="${90.0*M_PI/180}" />
     </joint>
     <link name="l_pinky0">
@@ -360,5 +370,6 @@
     <joint name="left_hand_j10" type="revolute">
       <axis xyz="0 1 0" />
-      <limit effort="100" velocity="${1600*M_PI/180}" lower="${-34.99*M_PI/180}" upper="${34.99*M_PI/180}" />
+      <!--limit effort="100" velocity="${1600*M_PI/180}" lower="${-34.99*M_PI/180}" upper="${34.99*M_PI/180}" /-->
+	  <limit effort="100" velocity="${1600*M_PI/180}" lower="${-7.072*M_PI/180}" upper="${90.0*M_PI/180}" />
       <origin xyz="0 0 -0.044" rpy="0 0 0" />
       <parent link="l_pinky0"/>
@@ -391,5 +402,6 @@
     <joint name="left_hand_j11" type="revolute">
       <axis xyz="0 1 0" />
-      <limit effort="100" velocity="${1600*M_PI/180}" lower="${-34.21*M_PI/180}" upper="${34.213*M_PI/180}" />
+      <!--limit effort="100" velocity="${1600*M_PI/180}" lower="${-34.21*M_PI/180}" upper="${34.213*M_PI/180}" /-->
+	  <limit effort="100" velocity="${1600*M_PI/180}" lower="${-7.072*M_PI/180}" upper="${90.0*M_PI/180}" />
       <origin xyz="0 0 -0.032" rpy="0 0 0" />
       <parent link="l_pinky1"/>

File: gt_meka_description/urdf/H2R4_r_hand_defs.urdf.xacro (robot description, xacro)
@@ -55,5 +55,6 @@
       <parent link="palm"/>
       <child link="thumb0"/>
-      <limit effort="100" velocity="${20.0*M_PI/180}" lower="${-40*M_PI/180}" upper="${15*M_PI/180}" />
+      <!--limit effort="100" velocity="${20.0*M_PI/180}" lower="${-40*M_PI/180}" upper="${15*M_PI/180}" /-->
+      <limit effort="100" velocity="${20.0*M_PI/180}" lower="${0.7*M_PI/180}" upper="${90*M_PI/180}" />
     </joint>
     <link name="thumb0">
